File: Untitled.kicad 2_pcb.kicad_pcb (KiCad board)
At the start: 2 copper layers, 37 x 37 mm, 22 parts, among them J1 Battery Connector, J2 Top Screw Terminal, J3 Bottom Screw Terminal, Q1 Q_NMOS_DGS, Q2 Q_NMOS_DGS, Q3 Q_NMOS_DGS, U1 XIAO-ESP32-S3-SMD, U3 LSM6DSO32, U4 MS5611-01BA

Commit message: My PCB design
I arranged the parts and then used an automatic routing thingy to attach all of the nodes. I then made sure it followed the design rules checker and that's it.
Parts:
- J3: moved to F.Cu
- moved J3 0.27 mm to (214.0, 77.0)
Routing:
- net -BATT: track 86.9 -> 94.0 mm
- net /APPO: track 31.9 -> 38.3 mm
- net /MAIN: track 31.3 -> 25.4 mm, vias 2 -> 0
- net /SCL: track 20.7 -> 15.9 mm, vias 1 -> 0
- net /IGNIT 1: track 16.5 -> 13.3 mm
- net +3.3V: track 77.9 -> 80.7 mm, vias 0 -> 1
- net /MOTOR: track 26.8 -> 25.2 mm, vias 2 -> 1
- net /CONT 3: track 14.5 -> 15.7 mm
- net /CONT 2: track 31.4 -> 30.7 mm
- net /CONT 1: track 12.8 -> 12.2 mm, vias 1 -> 0
- net /IGNIT 3: track 11.0 -> 10.5 mm, vias 1 -> 0
- net +BATT: track 24.0 -> 24.2 mm, vias 0 -> 1
Other:
- board text removed: "JA"
- board text removed: "UCRC"
